File: pwr-bl-tch.kicad_sch (KiCad schematic)
At the start: 44 parts, among them J3 39 POS FFC(0.3mm), J5 Raspberry_Pi_GPIO, U1 TLV75733PDBV, U2 TLV75718PDBV, U3 TPS92380, U4 SN74LV1T34DBV, U5 TXS0104EPW

Commit message: Added missing BOM fileds for L1 and J5. Fixed L1 label on silk
Signed-off-by: Akshay Athalye <akshay@scandent.com>
Parts:
- J5: Manufacturer (none) -> Adafruit; Mfg. Part No. (none) -> 2222
- L1: Manufacturer (none) -> Pulse Electronics; Mfg. Part No. (none) -> BMRF00060630100MA1
Changed lines of the file:
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@@
 			)
 		)
-		(property "Description" "Inductor, small symbol"
+		(property "Description" "10UH 4A 68 MOHM"
 			(at 153.67 22.86 0)
 			(effects
@@
 			)
 		)
-		(property "Manufacturer" ""
+		(property "Manufacturer" "Pulse Electronics"
 			(at 153.67 22.86 90)
 			(effects
@@
 			)
 		)
-		(property "Mfg. Part No." ""
+		(property "Mfg. Part No." "BMRF00060630100MA1"
 			(at 153.67 22.86 90)
 			(effects
@@
 			)
 		)
-		(property "Description" "Raspberry Pi GPIO socket"
+		(property "Description" "GPIO FEMALE HEADER  PI"
 			(at 89.408 128.778 0)
 			(effects
@@
 			)
 		)
-		(property "Manufacturer" ""
+		(property "Manufacturer" "Adafruit"
 			(at 73.66 99.06 0)
 			(effects
@@
 			)
 		)
-		(property "Mfg. Part No." ""
+		(property "Mfg. Part No." "2222"
 			(at 73.66 99.06 0)
 			(effects
