File: tv070hat.kicad_pcb (KiCad board)
At the start: 4 copper layers, 56.5 x 65 mm, 54 parts, among them J2 22Pos FFC(0.5mm), J3 39 POS FFC(0.3mm), J5 Raspberry_Pi_GPIO, U1 TLV75733PDBV, U2 TLV75718PDBV, U3 TPS92380, U4 SN74LV1T34DBV, U5 TXS0104EPW, U6 SN74LV1T34DBV, U7 HAT_Outline

Commit message: Added missing BOM fileds for L1 and J5. Fixed L1 label on silk
Signed-off-by: Akshay Athalye <akshay@scandent.com>
Changed lines of the file:
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@@
 		(at 139.567158 94.077545 -90)
 		(property "Reference" "L1"
-			(at 0 -0.5 270)
+			(at 0.322455 4.467158 270)
 			(unlocked yes)
-			(layer "F.Fab")
+			(layer "F.SilkS")
 			(effects
 				(font
